Commit message: Control the servos, send the command from ROS moveit and do the planning with ROS moveit.
Action server to keep communication with robot
ros2 run my_robot_first_servo_control servo_client

Action server client for sending the angles and listening to joint_state from moveit
ros2 run my_robot_first_servo_control servo_client_client

To start the RVIZ and movit
ros2 launch myrobot_moveit_config myrobot_planning_execution.launch.py
To move the robot to another position with moveit
ros2 run myrobot_hello_moveit myrobot_hello_moveit

File: install/myrobot_moveit_config/share/myrobot_moveit_config/config/arm_base.xacro (robot description, xacro)
@@ -115,7 +115,7 @@
         <collision>
             <geometry>
-                <box size="${link4_length} ${link4_width} ${link4_height}" />
-            </geometry>
-            <origin xyz="${link4_width/2.0} ${link4_height/2.0} 0" rpy="1.5708 0 0" />
+                <box size="${link4_length} ${link4_width} ${link4_height*0.8}" />
+            </geometry>
+            <origin xyz="${link4_width/2.0} ${link4_height/1.6} 0" rpy="1.5708 0 0" />
         </collision>
         <xacro:box_inertia m="0.5" l="${2*link4_length}" w="${2*link4_width}" h="${2*link4_height}"
