Commit message: Added an improved URDF and hello world program where now I can find the range of the robot movements which will help me get the better positions and orientations

File: install/moveit_resources_dragon_description/share/moveit_resources_dragon_description/urdf/dragon.urdf (robot description, URDF)
Before this commit: robot dragon_model, 8 links, 7 joints
Links:
- removed link Left_finger_link
- removed link Right_finger_link
- removed link servo2_servo3_link.000
- added link left_finger_link; collision mesh filename=package://moveit_resources_dragon_description/meshes/stl/le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 scale=0.001 0.001 0.001; visual mesh filename=package://moveit_resources_dragon_description/meshes/stl/le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 scale=0.001 0.001 0.001
- added link right_finger_link; collision mesh filename=package://moveit_resources_dragon_description/meshes/stl/ri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 scale=0.001 0.001 0.001; visual mesh filename=package://moveit_resources_dragon_description/meshes/stl/ri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 scale=0.001 0.001 0.001
- added link servo2_servo3_link; collision mesh filename=package://moveit_resources_dragon_description/meshes/stl/jo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 scale=0.001 0.001 0.001; visual mesh filename=package://moveit_resources_dragon_description/meshes/stl/jo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 scale=0.001 0.001 0.001
- link base_link: geometry collision mesh filename=package://moveit_resources_dragon_description/meshes/stl/ba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 scale=0.001 0.001 0.001; visual mesh filename=package://moveit_resources_dragon_description/meshes/stl/ba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 scale=0.001 0.001 0.001
- link servo1_servo2_link: geometry collision mesh filename=package://moveit_resources_dragon_description/meshes/stl/jo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 scale=0.001 0.001 0.001; visual mesh filename=package://moveit_resources_dragon_description/meshes/stl/jo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 scale=0.001 0.001 0.001
- link servo3_servo4_link: geometry collision mesh filename=package://moveit_resources_dragon_description/meshes/stl/jo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 scale=0.001 0.001 0.001; visual mesh filename=package://moveit_resources_dragon_description/meshes/stl/jo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 scale=0.001 0.001 0.001
- link servo4_servo5_link: geometry collision mesh filename=package://moveit_resources_dragon_description/meshes/stl/jo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 scale=0.001 0.001 0.001; visual mesh filename=package://moveit_resources_dragon_description/meshes/stl/jo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 scale=0.001 0.001 0.001
- link servo5_servo6_link: geometry collision mesh filename=package://moveit_resources_dragon_description/meshes/stl/gr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 scale=0.001 0.001 0.001; visual mesh filename=package://moveit_resources_dragon_description/meshes/stl/gr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 scale=0.001 0.001 0.001
Joints:
- removed joint servo1_servo2_link_joint
- removed joint servo2_servo3_link.000_joint
- removed joint servo3_servo4_link_joint
- removed joint servo4_servo5_link_joint
- removed joint wrist_link_joint
- added joint joint1: type revolute, parent base_link, child servo1_servo2_link, origin xyz=0.0 0.0 0.127335 rpy=0.00000000 0.00000000 -1.57079637, axis 0.00000000 0.00000000 1.00000000, limit lower=0.00000000 upper=3.14199996 effort=87 velocity=2.3925
- added joint joint2: type revolute, parent servo1_servo2_link, child servo2_servo3_link, origin xyz=0.0 0.0 0.016674 rpy=-1.57079637 0.00000000 0.00000000, axis 0.00000000 0.00000000 1.00000000, limit lower=0.00000000 upper=3.14000010 effort=87 velocity=2.3925
- added joint joint3: type revolute, parent servo2_servo3_link, child servo3_servo4_link, origin xyz=-0.104538 0.0 -0.00000006 rpy=3.14159265 0.00000000 3.14159257, axis 0.00000000 0.00000000 1.00000000, limit lower=0.00000000 upper=3.14000010 effort=87 velocity=2.3925
- added joint joint4: type revolute, parent servo3_servo4_link, child servo4_servo5_link, origin xyz=-0.008356 -0.101547 0.00001584 rpy=3.14159257 -0.00000012 0.00000000, axis 0.00000000 0.00000000 1.00000000, limit lower=0.00000000 upper=3.14000010 effort=87 velocity=2.3925
- added joint joint5: type revolute, parent servo4_servo5_link, child servo5_servo6_link, origin xyz=-0.028738 0.047654 0.00000208 rpy=-1.57079628 -0.00000009 0.00000009, axis 0.00000000 0.00000000 1.00000000, limit lower=0.00000000 upper=3.14000010 effort=87 velocity=2.3925
- joint left_hand_finger_joint: axis 0 -1 0 -> 0 0 1; child Left_finger_link -> left_finger_link; origin xyz=0.00121974 0.02889340 -0.00150631 rpy=-1.57080 0.00000 0.00000 -> xyz=0.000101 -0.000827 0.057582 rpy=1.57079637 0.00000000 -3.14159257
- joint right_hand_finger_joint: axis 0 1 0 -> 0 0 -1; child Right_finger_link -> right_finger_link; origin xyz=0.00121974 0.02889340 -0.00150631 rpy=-1.57080 0.00000 0.00000 -> xyz=0.000101 -0.000827 0.057582 rpy=1.57079637 0.00000000 -3.14159257

Commit message: Now I can make the robot move with rviz and the reality matches with it. Next step is move to camera calibration

File: install/moveit_resources_dragon_description/share/moveit_resources_dragon_description/urdf/dragon.urdf (robot description, URDF)
Before this commit: robot 6DoF, 8 links, 7 joints
Joints:
- joint joint4: axis 0.00000000 0.00000000 1.00000000 -> 0.00000000 0.00000000 -1.00000000
